File: CC1310_7X7 SubGHz/cc1310_7x7.sch (KiCad schematic (older format))
At the start: 63 parts, among them P1 CONN_02X03, P2 XBEE, P3 JTAG, SW1 RESET, SW2 USER_BUTTON, U1 cc1310_7x7, U2 LTR-303ALS, U3 Si7006, U6 SMA_EDGE_CONNECTOR, Y1 32.768 KHz, Y2 crystal

Commit message: modified inductor library; added inductor in schematic
Parts:
- removed L3, L4: 7.5nH, symbol INDUCTOR
- added L3, L4: 7.5nH, symbol inductor
Other:
- note removed: "."
- moved on the sheet: C19
Changed lines of the file:
@@
 L C C19
 U 1 1 582F437F
-P 6900 7800
-F 0 "C19" H 6925 7900 50  0000 L CNN
-F 1 "100pF" H 6925 7700 50  0000 L CNN
-F 2 "" H 6938 7650 50  0000 C CNN
-F 3 "" H 6900 7800 50  0000 C CNN
-	1    6900 7800
+P 6900 8150
+F 0 "C19" H 6925 8250 50  0000 L CNN
+F 1 "100pF" H 6925 8050 50  0000 L CNN
+F 2 "" H 6938 8000 50  0000 C CNN
+F 3 "" H 6900 8150 50  0000 C CNN
+	1    6900 8150
 	1    0    0    -1
 $EndComp
@@
 L GND #PWR21
 U 1 1 582F479C
-P 6900 8000
-F 0 "#PWR21" H 6900 7750 50  0001 C CNN
-F 1 "GND" H 6900 7850 50  0000 C CNN
-F 2 "" H 6900 8000 50  0000 C CNN
-F 3 "" H 6900 8000 50  0000 C CNN
-	1    6900 8000
+P 6900 8350
+F 0 "#PWR21" H 6900 8100 50  0001 C CNN
+F 1 "GND" H 6900 8200 50  0000 C CNN
+F 2 "" H 6900 8350 50  0000 C CNN
+F 3 "" H 6900 8350 50  0000 C CNN
+	1    6900 8350
 	1    0    0    -1
 $EndComp
@@
 	1    8400 6000
 	0    -1   -1   0
-$EndComp
-$Comp
-L INDUCTOR L4
-U 1 1 582FAD41
-P 7200 6000
-F 0 "L4" V 7350 6000 50  0000 C CNN
-F 1 "7.5nH" V 7100 6000 50  0000 C CNN
-F 2 "" H 7200 6000 50  0000 C CNN
-F 3 "" H 7200 6000 50  0000 C CNN
-	1    7200 6000
-	0    -1   -1   0
-$EndComp
-$Comp
-L INDUCTOR L3
-U 1 1 582FB1F5
-P 6900 7200
-F 0 "L3" H 7050 7250 50  0000 C CNN
-F 1 "7.5nH" H 7100 7100 50  0000 C CNN
-F 2 "" H 6900 7200 50  0000 C CNN
-F 3 "" H 6900 7200 50  0000 C CNN
-	1    6900 7200
-	1    0    0    -1
 $EndComp
 Text GLabel 5200 5500 1    39   Input ~ 0
@@
 	0    1    1    0
 $EndComp
-Text Notes 6850 7100 0    197  ~ 0
-.
-Text Notes 7000 6050 0    197  ~ 0
-.
 $Comp
 L Crystal Y1
@@
 	5000 2875 5000 3175
 Wire Wire Line
-	6900 7400 6900 7650
+	6900 7700 6900 8000
 Wire Wire Line
 	6750 5450 6450 5450
@@
 	5900 7050 6550 7050
 Wire Wire Line
-	6550 7050 6550 7550
-Wire Wire Line
-	6550 7550 6900 7550
-Connection ~ 6900 7550
+	6550 7050 6550 7900
+Wire Wire Line
+	6550 7900 6900 7900
+Connection ~ 6900 7900
 Wire Wire Line
 	2800 6600 2100 6600
@@
 	1800 10100 1800 10150
 Wire Wire Line
-	6100 6000 6900 6000
-Wire Wire Line
 	6100 6700 6100 6800
 Wire Wire Line
@@
 Connection ~ 7950 6000
 Wire Wire Line
-	7500 6000 8100 6000
-Wire Wire Line
 	8700 6000 9000 6000
 Wire Wire Line
@@
 	5350 8225 5350 8150
 Wire Wire Line
-	6900 7950 6900 8000
+	6900 8300 6900 8350
 Wire Notes Line
 	15975 8150 12600 8150
@@
 	1    0    0    -1
 $EndComp
+$Comp
+L inductor L4
+U 1 1 5833FD1D
+P 7050 7100
+F 0 "L4" V 7325 7200 60  0000 C CNN
+F 1 "7.5nH" H 7250 6850 60  0000 C CNN
+F 2 "" H 7050 7100 60  0001 C CNN
+F 3 "" H 7050 7100 60  0001 C CNN
+	1    7050 7100
+	0    1    1    0
+$EndComp
+$Comp
+L inductor L3
+U 1 1 58343989
+P 7025 5850
+F 0 "L3" H 7250 5900 60  0000 C CNN
+F 1 "7.5nH" H 7225 5625 60  0000 C CNN
+F 2 "" H 7025 5850 60  0001 C CNN
+F 3 "" H 7025 5850 60  0001 C CNN
+	1    7025 5850
+	1    0    0    -1
+$EndComp
+Wire Wire Line
+	7625 6000 8100 6000
+Wire Wire Line
+	6100 6000 6825 6000
 $EndSCHEMATC

Commit message: initial design ready; modified JTAG, LTR303, TPS63051
Parts:
- added C29, C31, C32: 10uF, symbol C
- added C30: 1nF, symbol C
- added L7: 1.5uH, symbol INDUCTOR
- added R13: 0E, symbol R
- added R14: DNM, symbol R
- added R15: 100K, symbol R
- added R16: DNM, symbol R_Small
- added U4: TPS63051, symbol TPS63051
- D2: value ORANGE -> YELLOW
- D3: value YELLOW -> GREEN
- D4: value GREEN -> ORANGE
Connections:
- net labels added: CC1310_VIN, STAT, VOUT_XBEE
- net labels removed: +3V3, DIO_1
- wire segments 208 -> 240
Other:
- note added: "TPS63051 Single Inductor Buck-Boost With 1-A Switches\nVin = 2.5 V to 5.5 V\nVout = 3.3 V\nIout = 500 mA (boost mode) or 1 A (buck mode)"
- moved on the sheet: C11, C12, C13, C16, C18, C21, C22, C4, C6, C8, C9, FL1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

Commit message: modified TPS782 lib; added optional power section; ready for verification
Parts:
- removed R16: DNM, symbol R_Small
- added C? (x2): 1uF, symbol C
- added U?: TPS782, symbol TPS782
Connections:
- net labels added: DIO_1
- net labels removed: STAT
- wire segments 240 -> 250
Other:
- note added: "OPTIONAL POWER Section"
- moved on the sheet: C1, C14, C15, C17, C19, C2, C20, C23, C24, C25, C26, C27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

Commit message: re annotated the schematic
Parts:
- gave numbers to parts that had none: 3
- renumbered C29 to C1, C4 to C11, C6 to C12, C14 to C13, C8 to C14, C9 to C16, C11 to C17, C17 to C18, C1 to C2, C12 to C20, C20 to C21, C13 to C22, C16 to C25, C18 to C26, C25 to C27, C21 to C28, C26 to C29, C2 to C3, C27 to C30, C22 to C31, C28 to C32, C3 to C4, C7 to C5, C30 to C6, C5 to C7, C31 to C8, C32 to C9, L7 to L1, L1 to L6, L6 to L7, P3 to P2, P2 to P3, R9 to R10, R13 to R11, R8 to R12, R10 to R13, R11 to R14, R12 to R15, R4 to R3, R5 to R4, R3 to R5, R14 to R6, R6 to R7, R15 to R8, R7 to R9, U4 to U1, U1 to U2, U2 to U3, U3 to U4, U6 to U5
Other:
- note added: "Place L6 and C25 close to pin 33 (DCDC_SW)\nLow inductance ground for C25"
- note removed: "Place L1 and C16 close to pin 33 (DCDC_SW)\nLow inductance ground for C16"
